Commit message: Fixed publisher interference

File: WRORobot/urdf/wro_bot.urdf.xacro (robot description, xacro)
@@ -194,5 +194,5 @@
     <parent link="base_link"/>
     <child link="base_laser"/>
-    <origin xyz="${lidar_xyz}" rpy="0 0 0"/>
+    <origin xyz="${lidar_xyz}" rpy="0 0 -1.5708"/>
   </joint>
   <link name="imu_link">
