Commit message: working sim stack + pillar detector; open_challenge WIP

File: WRORobot/urdf/wro_bot.urdf.xacro (robot description, xacro)
@@ -25,12 +25,21 @@
   <xacro:property name="chassis_height" value="0.14"/>
   <!-- Sensor mount offsets (all in base_link frame). -->
-  <!-- TODO(measure): lidar mount position on real bot -->
-  <xacro:property name="lidar_xyz" value="0.0 0.05 0.07"/>
+  <!-- TODO(measure): lidar mount position on real bot.
+       Target: 8.5 cm above ground. base_link sits at world z = 0.103
+       (= wheel_radius + chassis_height/2), so world 0.085 = base_link
+       offset -0.018.
+       WARNING: with the current placeholder chassis_height (0.14 m), this
+       Z sits inside the chassis collision box and will produce self-hits
+       (0.13-0.16 m returns on every ray). Shrink chassis_height to a
+       realistic WRO value (~0.05 m) before trusting scans. -->
+  <xacro:property name="lidar_xyz" value="0.0 0.05 -0.018"/>
   <!-- TODO(measure): IMU mount position on real bot -->
   <xacro:property name="imu_xyz" value="0.0 0.09 0.10"/>
   <!-- TODO(measure): camera mount position on real bot (front-facing).
-       Component numbers to keep this trivially editable — camera lives at
-       (chassis_length/2 - 0.01, 0.0, 0.06). -->
-  <xacro:property name="camera_x" value="0.14"/>
+       camera_x must clear the chassis front face (chassis_length/2 = 0.14)
+       plus the camera body half-depth (~0.01). Sitting camera at exactly
+       chassis_length/2 puts the sensor inside the chassis geometry and
+       renders a blank/single-color image. -->
+  <xacro:property name="camera_x" value="0.16"/>
   <xacro:property name="camera_y" value="0.0"/>
   <xacro:property name="camera_z" value="0.06"/>

Commit message: changed orientation for lidar

File: WRORobot/urdf/wro_bot.urdf.xacro (robot description, xacro)
@@ -194,5 +194,5 @@
     <parent link="base_link"/>
     <child link="base_laser"/>
-    <origin xyz="${lidar_xyz}" rpy="0 0 0"/>
+    <origin xyz="${lidar_xyz}" rpy="0 0 1.5708"/>
   </joint>
   <link name="imu_link">

Commit message: changed the yaw (or x axis rotation) to -90 in radians

File: WRORobot/urdf/wro_bot.urdf.xacro (robot description, xacro)
@@ -194,5 +194,5 @@
     <parent link="base_link"/>
     <child link="base_laser"/>
-    <origin xyz="${lidar_xyz}" rpy="0 0 1.5708"/>
+    <origin xyz="${lidar_xyz}" rpy="0 0 0"/>
   </joint>
   <link name="imu_link">

Commit message: saftey chatch fix

File: WRORobot/urdf/wro_bot.urdf.xacro (robot description, xacro)
@@ -17,5 +17,5 @@
   <xacro:property name="wheel_radius" value="0.033"/>
   <!-- TODO(measure): tire width -->
-  <xacro:property name="wheel_thickness" value="0.025"/>
+  <xacro:property name="wheel_thickness" value="0.028"/>
   <!-- TODO(measure): mechanical max steer of the front wheels (30 deg) -->
   <xacro:property name="max_steer_angle" value="0.5236"/>
@@ -23,5 +23,5 @@
   <xacro:property name="chassis_length" value="0.28"/>
   <xacro:property name="chassis_width" value="0.16"/>
-  <xacro:property name="chassis_height" value="0.14"/>
+  <xacro:property name="chassis_height" value="0.19"/>
   <!-- Sensor mount offsets (all in base_link frame). -->
   <!-- TODO(measure): lidar mount position on real bot.
@@ -43,7 +43,9 @@
        chassis_length/2 puts the sensor inside the chassis geometry and
        renders a blank/single-color image. -->
-  <xacro:property name="camera_x" value="0.16"/>
+  <xacro:property name="camera_x" value="0.2162"/>
   <xacro:property name="camera_y" value="0.0"/>
-  <xacro:property name="camera_z" value="0.06"/>
+  <xacro:property name="camera_z" value="0.0466"/>
+  <!-- Camera pitch: negative = looking down (WRO block detection). -->
+  <xacro:property name="camera_pitch" value="${-20 * pi / 180}"/>
   <!-- Derived. -->
   <xacro:property name="half_l" value="${wheelbase/2}"/>
@@ -217,5 +219,5 @@
     <parent link="base_link"/>
     <child link="camera_link"/>
-    <origin xyz="${camera_x} ${camera_y} ${camera_z}" rpy="0 0 0"/>
+    <origin xyz="${camera_x} ${camera_y} ${camera_z}" rpy="0 ${camera_pitch} 0"/>
   </joint>
   <!-- ROS image convention frame (Z forward, X right, Y down). Attach the

Commit message: new loop nav

File: WRORobot/urdf/wro_bot.urdf.xacro (robot description, xacro)
@@ -33,7 +33,7 @@
        (0.13-0.16 m returns on every ray). Shrink chassis_height to a
        realistic WRO value (~0.05 m) before trusting scans. -->
-  <xacro:property name="lidar_xyz" value="0.0 0.05 -0.018"/>
+  <xacro:property name="lidar_xyz" value="0.0 0.05 ${-0.018 + chassis_z}"/>
   <!-- TODO(measure): IMU mount position on real bot -->
-  <xacro:property name="imu_xyz" value="0.0 0.09 0.10"/>
+  <xacro:property name="imu_xyz" value="0.0 0.09 ${0.10 + chassis_z}"/>
   <!-- TODO(measure): camera mount position on real bot (front-facing).
        On the real bot this is the Limelight 3's front mount; in sim it's
@@ -67,7 +67,7 @@
        Reusable macros.
        ============================================================ -->
-  <xacro:macro name="inertial_box" params="mass x y z">
+  <xacro:macro name="inertial_box" params="mass x y z offset_z:=0">
     <inertial>
-      <origin xyz="0 0 0" rpy="0 0 0"/>
+      <origin xyz="0 0 ${offset_z}" rpy="0 0 0"/>
       <mass value="${mass}"/>
       <inertia
@@ -116,5 +116,5 @@
   <link name="base_link">
     <visual>
-      <origin xyz="0 0 0" rpy="0 0 0"/>
+      <origin xyz="0 0 ${chassis_z}" rpy="0 0 0"/>
       <geometry>
         <box size="${chassis_length} ${chassis_width} ${chassis_height}"/>
@@ -123,10 +123,10 @@
     </visual>
     <collision>
-      <origin xyz="0 0 0" rpy="0 0 0"/>
+      <origin xyz="0 0 ${chassis_z}" rpy="0 0 0"/>
       <geometry>
         <box size="${chassis_length} ${chassis_width} ${chassis_height}"/>
       </geometry>
     </collision>
-    <xacro:inertial_box mass="1.5" x="${chassis_length}" y="${chassis_width}" z="${chassis_height}"/>
+    <xacro:inertial_box mass="1.5" x="${chassis_length}" y="${chassis_width}" z="${chassis_height}" offset_z="${chassis_z}"/>
   </link>
   <!-- Steering knuckles (front left, front right). -->
@@ -140,5 +140,5 @@
     <parent link="base_link"/>
     <child link="front_left_wheel_steer"/>
-    <origin xyz="${half_l} ${half_t} ${-chassis_height/2}" rpy="0 0 0"/>
+    <origin xyz="${half_l} ${half_t} ${-chassis_height/2 + chassis_z}" rpy="0 0 0"/>
     <axis xyz="0 0 1"/>
     <limit lower="${-max_steer_angle}" upper="${max_steer_angle}"
@@ -148,5 +148,5 @@
     <parent link="base_link"/>
     <child link="front_right_wheel_steer"/>
-    <origin xyz="${half_l} ${-half_t} ${-chassis_height/2}" rpy="0 0 0"/>
+    <origin xyz="${half_l} ${-half_t} ${-chassis_height/2 + chassis_z}" rpy="0 0 0"/>
     <axis xyz="0 0 1"/>
     <limit lower="${-max_steer_angle}" upper="${max_steer_angle}"
@@ -173,5 +173,5 @@
     <parent link="base_link"/>
     <child link="rear_left_wheel"/>
-    <origin xyz="${-half_l} ${half_t} ${-chassis_height/2}" rpy="0 0 0"/>
+    <origin xyz="${-half_l} ${half_t} ${-chassis_height/2 + chassis_z}" rpy="0 0 0"/>
     <axis xyz="0 1 0"/>
   </joint>
@@ -179,5 +179,5 @@
     <parent link="base_link"/>
     <child link="rear_right_wheel"/>
-    <origin xyz="${-half_l} ${-half_t} ${-chassis_height/2}" rpy="0 0 0"/>
+    <origin xyz="${-half_l} ${-half_t} ${-chassis_height/2 + chassis_z}" rpy="0 0 0"/>
     <axis xyz="0 1 0"/>
   </joint>
@@ -219,5 +219,5 @@
     <parent link="base_link"/>
     <child link="camera_link"/>
-    <origin xyz="${camera_x} ${camera_y} ${camera_z}" rpy="0 ${camera_pitch} 0"/>
+    <origin xyz="${camera_x} ${camera_y} ${camera_z + chassis_z}" rpy="0 ${camera_pitch} 0"/>
   </joint>
   <!-- ROS image convention frame (Z forward, X right, Y down). Attach the

Commit message: nav 2 path

File: WRORobot/urdf/wro_bot.urdf.xacro (robot description, xacro)
@@ -23,5 +23,5 @@
   <xacro:property name="chassis_length" value="0.28"/>
   <xacro:property name="chassis_width" value="0.16"/>
-  <xacro:property name="chassis_height" value="0.19"/>
+  <xacro:property name="chassis_height" value="0.085"/>
   <!-- Sensor mount offsets (all in base_link frame). -->
   <!-- TODO(measure): lidar mount position on real bot.
@@ -33,7 +33,7 @@
        (0.13-0.16 m returns on every ray). Shrink chassis_height to a
        realistic WRO value (~0.05 m) before trusting scans. -->
-  <xacro:property name="lidar_xyz" value="0.0 0.05 ${-0.018 + chassis_z}"/>
+  <xacro:property name="lidar_xyz" value="0.0 0.05 ${0.085-chassis_z}"/>
   <!-- TODO(measure): IMU mount position on real bot -->
-  <xacro:property name="imu_xyz" value="0.0 0.09 ${0.10 + chassis_z}"/>
+  <xacro:property name="imu_xyz" value="0.0 0.00 0.01"/>
   <!-- TODO(measure): camera mount position on real bot (front-facing).
        On the real bot this is the Limelight 3's front mount; in sim it's
@@ -43,9 +43,9 @@
        chassis_length/2 puts the sensor inside the chassis geometry and
        renders a blank/single-color image. -->
-  <xacro:property name="camera_x" value="0.2162"/>
+  <xacro:property name="camera_x" value="0.02162"/>
   <xacro:property name="camera_y" value="0.0"/>
   <xacro:property name="camera_z" value="0.0466"/>
   <!-- Camera pitch: negative = looking down (WRO block detection). -->
-  <xacro:property name="camera_pitch" value="${-20 * pi / 180}"/>
+  <xacro:property name="camera_pitch" value="${-pi/9}"/>
   <!-- Derived. -->
   <xacro:property name="half_l" value="${wheelbase/2}"/>
@@ -67,7 +67,7 @@
        Reusable macros.
        ============================================================ -->
-  <xacro:macro name="inertial_box" params="mass x y z offset_z:=0">
+  <xacro:macro name="inertial_box" params="mass x y z">
     <inertial>
-      <origin xyz="0 0 ${offset_z}" rpy="0 0 0"/>
+      <origin xyz="0 0 0" rpy="0 0 0"/>
       <mass value="${mass}"/>
       <inertia
@@ -116,5 +116,5 @@
   <link name="base_link">
     <visual>
-      <origin xyz="0 0 ${chassis_z}" rpy="0 0 0"/>
+      <origin xyz="0 0 0" rpy="0 0 0"/>
       <geometry>
         <box size="${chassis_length} ${chassis_width} ${chassis_height}"/>
@@ -123,10 +123,10 @@
     </visual>
     <collision>
-      <origin xyz="0 0 ${chassis_z}" rpy="0 0 0"/>
+      <origin xyz="0 0 0" rpy="0 0 0"/>
       <geometry>
         <box size="${chassis_length} ${chassis_width} ${chassis_height}"/>
       </geometry>
     </collision>
-    <xacro:inertial_box mass="1.5" x="${chassis_length}" y="${chassis_width}" z="${chassis_height}" offset_z="${chassis_z}"/>
+    <xacro:inertial_box mass="1.5" x="${chassis_length}" y="${chassis_width}" z="${chassis_height}"/>
   </link>
   <!-- Steering knuckles (front left, front right). -->
@@ -140,5 +140,5 @@
     <parent link="base_link"/>
     <child link="front_left_wheel_steer"/>
-    <origin xyz="${half_l} ${half_t} ${-chassis_height/2 + chassis_z}" rpy="0 0 0"/>
+    <origin xyz="${half_l} ${half_t} ${-chassis_height/2}" rpy="0 0 0"/>
     <axis xyz="0 0 1"/>
     <limit lower="${-max_steer_angle}" upper="${max_steer_angle}"
@@ -148,5 +148,5 @@
     <parent link="base_link"/>
     <child link="front_right_wheel_steer"/>
-    <origin xyz="${half_l} ${-half_t} ${-chassis_height/2 + chassis_z}" rpy="0 0 0"/>
+    <origin xyz="${half_l} ${-half_t} ${-chassis_height/2}" rpy="0 0 0"/>
     <axis xyz="0 0 1"/>
     <limit lower="${-max_steer_angle}" upper="${max_steer_angle}"
@@ -173,5 +173,5 @@
     <parent link="base_link"/>
     <child link="rear_left_wheel"/>
-    <origin xyz="${-half_l} ${half_t} ${-chassis_height/2 + chassis_z}" rpy="0 0 0"/>
+    <origin xyz="${-half_l} ${half_t} ${-chassis_height/2}" rpy="0 0 0"/>
     <axis xyz="0 1 0"/>
   </joint>
@@ -179,5 +179,5 @@
     <parent link="base_link"/>
     <child link="rear_right_wheel"/>
-    <origin xyz="${-half_l} ${-half_t} ${-chassis_height/2 + chassis_z}" rpy="0 0 0"/>
+    <origin xyz="${-half_l} ${-half_t} ${-chassis_height/2}" rpy="0 0 0"/>
     <axis xyz="0 1 0"/>
   </joint>
@@ -219,5 +219,5 @@
     <parent link="base_link"/>
     <child link="camera_link"/>
-    <origin xyz="${camera_x} ${camera_y} ${camera_z + chassis_z}" rpy="0 ${camera_pitch} 0"/>
+    <origin xyz="${camera_x} ${camera_y} ${camera_z}" rpy="0 ${camera_pitch} 0"/>
   </joint>
   <!-- ROS image convention frame (Z forward, X right, Y down). Attach the

Commit message: new waypoint

File: WRORobot/urdf/wro_bot.urdf.xacro (robot description, xacro)
@@ -47,5 +47,5 @@
   <xacro:property name="camera_z" value="0.0466"/>
   <!-- Camera pitch: negative = looking down (WRO block detection). -->
-  <xacro:property name="camera_pitch" value="${-pi/9}"/>
+  <xacro:property name="camera_pitch" value="${pi/9}"/>
   <!-- Derived. -->
   <xacro:property name="half_l" value="${wheelbase/2}"/>

Commit message: open challenge sort of works

File: WRORobot/urdf/wro_bot.urdf.xacro (robot description, xacro)
@@ -107,11 +107,12 @@
   <!-- ============================================================
        Frames.
-       base_link is the tree root. The AckermannSteering plugin publishes
-       odom -> base_link on /model/wro_bot/tf; robot_state_publisher owns
-       every other transform. We do NOT define base_footprint (it would
-       give base_link two parents once the plugin's tf is bridged).
-       Spawn the model with z = wheel_radius + chassis_height/2 so wheels
-       touch the ground (see wro_sim/launch/gz_sim.launch.py 'z' default).
-       ============================================================ -->
+       base_footprint is the tree root — a virtual point on the ground
+       directly below base_link. The AckermannSteering plugin publishes
+       odom -> base_footprint on /model/wro_bot/tf; robot_state_publisher
+       owns base_footprint -> base_link and everything above.
+       Spawn the model with z = 0 — base_footprint is at ground level,
+       and the URDF lifts base_link by chassis_z internally.
+       ============================================================ -->
+  <link name="base_footprint"/>
   <link name="base_link">
     <visual>
@@ -130,4 +131,10 @@
     <xacro:inertial_box mass="1.5" x="${chassis_length}" y="${chassis_width}" z="${chassis_height}"/>
   </link>
+  <!-- Lift base_link (chassis centre) chassis_z above the ground plane. -->
+  <joint name="base_footprint_to_base_link" type="fixed">
+    <parent link="base_footprint"/>
+    <child link="base_link"/>
+    <origin xyz="0 0 ${chassis_z}" rpy="0 0 0"/>
+  </joint>
   <!-- Steering knuckles (front left, front right). -->
   <link name="front_left_wheel_steer">
@@ -259,5 +266,5 @@
       <tf_topic>/model/wro_bot/tf</tf_topic>
       <frame_id>odom</frame_id>
-      <child_frame_id>base_link</child_frame_id>
+      <child_frame_id>base_footprint</child_frame_id>
       <odom_publish_frequency>30</odom_publish_frequency>
     </plugin>
@@ -294,5 +301,5 @@
         </scan>
         <range>
-          <min>0.02</min>
+          <min>0.20</min>
           <max>8.0</max>
           <resolution>0.01</resolution>
