Commit message: new map for sim

File: wro_map_nav2_sim.sdf.xacro (robot description, xacro)
@@ -1,169 +1,665 @@
 <?xml version="1.0"?>
-<robot
-  xmlns:xacro="http://www.ros.org/wiki/xacro"
-  name="sft_arena">
-  <!-- ====================================================== -->
-  <!-- SETTINGS                                               -->
-  <!-- ====================================================== -->
-  <xacro:property name="floor_size" value="3.2"/>
-  <xacro:property name="wall_height" value="0.70"/>
-  <xacro:property name="wall_thickness" value="0.10"/>
-  <!-- Wall center is 1.55 m from the arena center -->
-  <xacro:property name="wall_position" value="1.55"/>
-  <!-- ====================================================== -->
-  <!-- COLORS                                                 -->
-  <!-- ====================================================== -->
-  <material name="floor_white">
-    <color rgba="0.95 0.95 0.95 1.0"/>
-  </material>
-  <material name="wall_grey">
-    <color rgba="0.70 0.70 0.70 1.0"/>
-  </material>
-  <!-- ====================================================== -->
-  <!-- ROOT                                                   -->
-  <!-- ====================================================== -->
-  <link name="sft_base"/>
-  <!-- ====================================================== -->
-  <!-- FLOOR / MAT                                            -->
-  <!--                                                        -->
-  <!-- Visual only: there is intentionally no collision here. -->
-  <!-- The normal Gazebo ground plane supports the robot.      -->
-  <!-- ====================================================== -->
-  <link name="world_mat">
-    <visual name="world_mat_visual">
-      <!--
-        The mat is 0.001 m thick.
-        Its top surface is at z = 0.
-      -->
-      <origin xyz="0 0 -0.0005" rpy="0 0 0"/>
-      <geometry>
-        <box size="3.2 3.2 0.001"/>
-      </geometry>
-      <material name="floor_white"/>
-    </visual>
-  </link>
-  <joint name="world_mat_joint" type="fixed">
-    <parent link="sft_base"/>
-    <child link="world_mat"/>
-    <origin xyz="0 0 0" rpy="0 0 0"/>
-  </joint>
-  <gazebo reference="world_mat">
-    <material>Gazebo/White</material>
-  </gazebo>
-  <!-- ====================================================== -->
-  <!-- NORTH WALL                                             -->
-  <!-- ====================================================== -->
-  <link name="north_wall">
-    <visual name="north_wall_visual">
-      <origin xyz="0 0 0" rpy="0 0 0"/>
-      <geometry>
-        <box size="3.2 0.10 0.70"/>
-      </geometry>
-      <material name="wall_grey"/>
-    </visual>
-    <collision name="north_wall_collision">
-      <origin xyz="0 0 0" rpy="0 0 0"/>
-      <geometry>
-        <box size="3.2 0.10 0.70"/>
-      </geometry>
-    </collision>
-  </link>
-  <joint name="north_wall_joint" type="fixed">
-    <parent link="sft_base"/>
-    <child link="north_wall"/>
-    <origin
-      xyz="0 ${wall_position} ${wall_height / 2.0}"
-      rpy="0 0 0"/>
-  </joint>
-  <gazebo reference="north_wall">
-    <material>Gazebo/Grey</material>
-  </gazebo>
-  <!-- ====================================================== -->
-  <!-- SOUTH WALL                                             -->
-  <!-- ====================================================== -->
-  <link name="south_wall">
-    <visual name="south_wall_visual">
-      <origin xyz="0 0 0" rpy="0 0 0"/>
-      <geometry>
-        <box size="3.2 0.10 0.70"/>
-      </geometry>
-      <material name="wall_grey"/>
-    </visual>
-    <collision name="south_wall_collision">
-      <origin xyz="0 0 0" rpy="0 0 0"/>
-      <geometry>
-        <box size="3.2 0.10 0.70"/>
-      </geometry>
-    </collision>
-  </link>
-  <joint name="south_wall_joint" type="fixed">
-    <parent link="sft_base"/>
-    <child link="south_wall"/>
-    <origin
-      xyz="0 -${wall_position} ${wall_height / 2.0}"
-      rpy="0 0 0"/>
-  </joint>
-  <gazebo reference="south_wall">
-    <material>Gazebo/Grey</material>
-  </gazebo>
-  <!-- ====================================================== -->
-  <!-- EAST WALL                                              -->
-  <!-- ====================================================== -->
-  <link name="east_wall">
-    <visual name="east_wall_visual">
-      <origin xyz="0 0 0" rpy="0 0 0"/>
-      <geometry>
-        <box size="0.10 3.2 0.70"/>
-      </geometry>
-      <material name="wall_grey"/>
-    </visual>
-    <collision name="east_wall_collision">
-      <origin xyz="0 0 0" rpy="0 0 0"/>
-      <geometry>
-        <box size="0.10 3.2 0.70"/>
-      </geometry>
-    </collision>
-  </link>
-  <joint name="east_wall_joint" type="fixed">
-    <parent link="sft_base"/>
-    <child link="east_wall"/>
-    <origin
-      xyz="${wall_position} 0 ${wall_height / 2.0}"
-      rpy="0 0 0"/>
-  </joint>
-  <gazebo reference="east_wall">
-    <material>Gazebo/Grey</material>
-  </gazebo>
-  <!-- ====================================================== -->
-  <!-- WEST WALL                                              -->
-  <!-- ====================================================== -->
-  <link name="west_wall">
-    <visual name="west_wall_visual">
-      <origin xyz="0 0 0" rpy="0 0 0"/>
-      <geometry>
-        <box size="0.10 3.2 0.70"/>
-      </geometry>
-      <material name="wall_grey"/>
-    </visual>
-    <collision name="west_wall_collision">
-      <origin xyz="0 0 0" rpy="0 0 0"/>
-      <geometry>
-        <box size="0.10 3.2 0.70"/>
-      </geometry>
-    </collision>
-  </link>
-  <joint name="west_wall_joint" type="fixed">
-    <parent link="sft_base"/>
-    <child link="west_wall"/>
-    <origin
-      xyz="-${wall_position} 0 ${wall_height / 2.0}"
-      rpy="0 0 0"/>
-  </joint>
-  <gazebo reference="west_wall">
-    <material>Gazebo/Grey</material>
-  </gazebo>
-  <!-- Make the complete arena immovable in Gazebo -->
-  <gazebo>
-    <static>true</static>
-  </gazebo>
-</robot>
+<sdf version="1.9"
+     xmlns:xacro="http://www.ros.org/wiki/xacro">
+  <!-- ================================================================
+       WRO FUTURE ENGINEERS 2026 FIELD
+       Intended for:
+         - ROS 2
+         - Gazebo Sim Harmonic or newer
+         - SDFormat 1.9
+       Units:
+         - metres
+         - kilograms
+         - radians
+       Generate with:
+         ros2 run xacro xacro \
+           wro_future_engineers_field.sdf.xacro \
+           -o wro_future_engineers_field.sdf
+       The official field dimensions represented here are:
+         Mat:                     3.200 x 3.200 m
+         Racetrack internal area: 3.000 x 3.000 m
+         Wall height:             0.100 m
+         Traffic sign:            0.050 x 0.050 x 0.100 m
+         Parking barrier:         0.200 x 0.020 x 0.100 m
+       Wall thickness is not defined by WRO.
+       This simulation uses 0.020 m by default.
+       IMPORTANT:
+       The traffic-sign and parking positions below are an example
+       obstacle layout. Change them to match your randomized round.
+       ================================================================ -->
+  <!-- ========================== ARGUMENTS ========================== -->
+  <!-- World -->
+  <xacro:arg name="world_name" default="wro_future_engineers"/>
+  <xacro:arg name="paused" default="false"/>
+  <!-- Open challenge: false; obstacle challenge: true -->
+  <xacro:arg name="with_obstacles" default="true"/>
+  <!-- Parking barriers -->
+  <xacro:arg name="with_parking" default="true"/>
+  <!--
+       Inner wall outside dimensions.
+       1.0 m inner wall gives approximately 1.0 m track corridors.
+       1.8 m inner wall gives approximately 0.6 m track corridors.
+       1.4 m is available for rectangular/randomized configurations.
+       Examples:
+         inner_x:=1.0 inner_y:=1.0
+         inner_x:=1.8 inner_y:=1.8
+         inner_x:=1.0 inner_y:=1.8
+         inner_x:=1.4 inner_y:=1.0
+  -->
+  <xacro:arg name="inner_x" default="1.0"/>
+  <xacro:arg name="inner_y" default="1.0"/>
+  <!-- WRO does not officially specify wall thickness -->
+  <xacro:arg name="wall_thickness" default="0.020"/>
+  <!-- Surface properties -->
+  <xacro:arg name="field_friction" default="0.80"/>
+  <xacro:arg name="field_friction2" default="0.80"/>
+  <!--
+       Set true after installing:
+       model://wro_future_engineers_field/materials/textures/wro_fe_2026_mat.png
+  -->
+  <xacro:arg name="use_mat_texture" default="false"/>
+  <!-- ========================== PROPERTIES ========================= -->
+  <xacro:property name="WORLD_NAME" value="$(arg world_name)"/>
+  <xacro:property name="MAT_SIZE" value="3.2"/>
+  <xacro:property name="TRACK_SIZE" value="3.0"/>
+  <xacro:property name="WALL_HEIGHT" value="0.1"/>
+  <xacro:property name="WALL_T" value="$(arg wall_thickness)"/>
+  <xacro:property name="INNER_X" value="$(arg inner_x)"/>
+  <xacro:property name="INNER_Y" value="$(arg inner_y)"/>
+  <xacro:property name="SIGN_X" value="0.05"/>
+  <xacro:property name="SIGN_Y" value="0.05"/>
+  <xacro:property name="SIGN_Z" value="0.10"/>
+  <xacro:property name="PARKING_X" value="0.20"/>
+  <xacro:property name="PARKING_Y" value="0.02"/>
+  <xacro:property name="PARKING_Z" value="0.10"/>
+  <!-- =========================== MACROS ============================ -->
+  <!-- Static box used for walls and barriers -->
+  <xacro:macro name="static_box"
+               params="name x y z sx sy sz r g b a:=1.0">
+    <model name="${name}">
+      <static>true</static>
+      <pose>${x} ${y} ${z} 0 0 0</pose>
+      <link name="link">
+        <collision name="collision">
+          <geometry>
+            <box>
+              <size>${sx} ${sy} ${sz}</size>
+            </box>
+          </geometry>
+          <surface>
+            <friction>
+              <ode>
+                <mu>0.80</mu>
+                <mu2>0.80</mu2>
+              </ode>
+            </friction>
+            <contact>
+              <ode>
+                <kp>1000000</kp>
+                <kd>100</kd>
+                <max_vel>0.01</max_vel>
+                <min_depth>0.001</min_depth>
+              </ode>
+            </contact>
+          </surface>
+        </collision>
+        <visual name="visual">
+          <geometry>
+            <box>
+              <size>${sx} ${sy} ${sz}</size>
+            </box>
+          </geometry>
+          <material>
+            <ambient>${r} ${g} ${b} ${a}</ambient>
+            <diffuse>${r} ${g} ${b} ${a}</diffuse>
+            <specular>0.02 0.02 0.02 1</specular>
+            <pbr>
+              <metal>
+                <roughness>0.95</roughness>
+                <metalness>0.0</metalness>
+              </metal>
+            </pbr>
+          </material>
+        </visual>
+      </link>
+    </model>
+  </xacro:macro>
+  <!-- Visual-only line on the floor -->
+  <xacro:macro name="floor_line"
+               params="name x y yaw length width r g b">
+    <model name="${name}">
+      <static>true</static>
+      <pose>${x} ${y} 0.0015 0 0 ${yaw}</pose>
+      <link name="link">
+        <visual name="visual">
+          <geometry>
+            <box>
+              <size>${length} ${width} 0.001</size>
+            </box>
+          </geometry>
+          <material>
+            <ambient>${r} ${g} ${b} 1</ambient>
+            <diffuse>${r} ${g} ${b} 1</diffuse>
+            <specular>0 0 0 1</specular>
+          </material>
+        </visual>
+      </link>
+    </model>
+  </xacro:macro>
+  <!-- Movable traffic sign -->
+  <xacro:macro name="traffic_sign"
+               params="name x y colour">
+    <model name="${name}">
+      <static>false</static>
+      <!-- Bottom of the sign is at field level -->
+      <pose>${x} ${y} ${SIGN_Z / 2.0} 0 0 0</pose>
+      <link name="link">
+        <inertial>
+          <mass>0.10</mass>
+          <!-- Cuboid inertia for 0.05 x 0.05 x 0.10 m -->
+          <inertia>
+            <ixx>0.00010417</ixx>
+            <iyy>0.00010417</iyy>
+            <izz>0.00004167</izz>
+            <ixy>0</ixy>
+            <ixz>0</ixz>
+            <iyz>0</iyz>
+          </inertia>
+        </inertial>
+        <collision name="collision">
+          <geometry>
+            <box>
+              <size>${SIGN_X} ${SIGN_Y} ${SIGN_Z}</size>
+            </box>
+          </geometry>
+          <surface>
+            <friction>
+              <ode>
+                <mu>0.65</mu>
+                <mu2>0.65</mu2>
+              </ode>
+            </friction>
+            <contact>
+              <ode>
+                <kp>500000</kp>
+                <kd>50</kd>
+                <max_vel>0.02</max_vel>
+                <min_depth>0.001</min_depth>
+              </ode>
+            </contact>
+          </surface>
+        </collision>
+        <visual name="visual">
+          <geometry>
+            <box>
+              <size>${SIGN_X} ${SIGN_Y} ${SIGN_Z}</size>
+            </box>
+          </geometry>
+          <material>
+            <xacro:if value="${colour == 'red'}">
+              <!-- Official WRO RGB: 238, 39, 55 -->
+              <ambient>0.933 0.153 0.216 1</ambient>
+              <diffuse>0.933 0.153 0.216 1</diffuse>
+            </xacro:if>
+            <xacro:if value="${colour == 'green'}">
+              <!-- Official WRO RGB: 68, 214, 44 -->
+              <ambient>0.267 0.839 0.173 1</ambient>
+              <diffuse>0.267 0.839 0.173 1</diffuse>
+            </xacro:if>
+            <specular>0.02 0.02 0.02 1</specular>
+            <pbr>
+              <metal>
+                <roughness>0.90</roughness>
+                <metalness>0.0</metalness>
+              </metal>
+            </pbr>
+          </material>
+        </visual>
+      </link>
+    </model>
+  </xacro:macro>
+  <!-- Parking barrier -->
+  <xacro:macro name="parking_barrier"
+               params="name x y yaw">
+    <model name="${name}">
+      <static>true</static>
+      <pose>${x} ${y} ${PARKING_Z / 2.0} 0 0 ${yaw}</pose>
+      <link name="link">
+        <collision name="collision">
+          <geometry>
+            <box>
+              <size>${PARKING_X} ${PARKING_Y} ${PARKING_Z}</size>
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